File: joystick_pcb/joystick_pcb.kicad_pcb (KiCad board)
At the start: 2 copper layers, 30 x 30 mm, 7 parts, among them J1 Conn_01x06_Pin, J2 Conn_01x06_Pin, U1 RKJXV122400R

Commit message: updated
Parts:
- removed REF** (x4): MountingHole_3.2mm_M3, MountingHole:MountingHole_3.2mm_M3
- moved J1 1.03 mm to (22.5, 29.7)
- moved J2 1.03 mm to (47.9, 29.7)
- moved U1 0.94 mm to (35.2, 35.9)
Routing:
- net VCC: track 40.9 -> 20.5 mm
- net GND: track 54.2 -> 41.5 mm
- net SW2: track 31.0 -> 28.5 mm
Other:
- board size 30 x 30 mm -> 30.5 x 24.1 mm

Commit message: updated
Parts:
- added REF**: MountingHole_3.5mm, MountingHole:MountingHole_3.5mm, F.Cu at (47.2, 24.0)
- added REF**: MountingHole_3.5mm, MountingHole:MountingHole_3.5mm, F.Cu at (23.2, 24.0)
- added REF**: MountingHole_3.5mm, MountingHole:MountingHole_3.5mm, F.Cu at (23.2, 48.0)
- added REF**: MountingHole_3.5mm, MountingHole:MountingHole_3.5mm, F.Cu at (47.2, 48.0)
Routing:
- net VCC: track 20.5 -> 50.8 mm
- net GND: track 41.5 -> 39.1 mm
Other:
- board size 30.5 x 24.1 mm -> 30 x 30 mm
